File: Hardware/EbookReader Board.brd (EAGLE design)
At the start: 170 x 111 mm, 103 parts, among them IC1 BD5229G-TR, IC4 XC6220A331MR-G, J1 FH34SRJ-24S-0.5SH_99_, J2 SAMACSYS_PARTS_USB4110-GF-A, J3 QWIIC_RIGHT_ANGLE, J4 112A-TAAR-R03_ATTEND, Q1 20V/4.2A/52mΩ/1.4W, Q2 20V/4.2A/52mΩ/1.4W, Q3 SI1308EDL-T1-GE3, U1 W25Q512JVEIQ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

Commit message: Modificari model 3D dispozitiv si PCB
Parts:
- moved TP7 68.4 mm to (95.3, 11.2)
- moved TP8 63.3 mm to (47.1, 35.7)
- moved TP15 58.4 mm to (108.1, 60.1)
- moved TP17 29.3 mm to (88.8, 21.1)
- moved TP6 26.7 mm to (34.3, 56.9)
- moved TP16 22.1 mm to (139.1, 43.1)
- moved TP14 17.0 mm to (111.3, 60.2)
- moved TP12 14.0 mm to (98.7, 11.0)
- moved D6 10.3 mm to (77.7, 23.3)
- moved TP4 10.0 mm to (28.3, 101.0)
- moved TP9 8.22 mm to (86.2, 21.1)
- moved R9 7.21 mm to (75.7, 22.3)
- moved TP1 7.00 mm to (3.27, 70.3)
- moved TP2 7.00 mm to (5.42, 70.2)
- moved TP10 6.00 mm to (82.1, 101.2)
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Routing:
- net SCK: track 201.8 -> 155.7 mm
- net INT_RTC: track 146.8 -> 117.1 mm, vias 4 -> 2
- net EPD_3V3: track 63.4 -> 35.7 mm, vias 2 -> 3
- net EPD_3V3_C: track 132.7 -> 158.3 mm, vias 4 -> 3
- net MISO: track 94.6 -> 115.5 mm, vias 4 -> 0
- net EPD_BUSY: track 124.0 -> 105.1 mm
- net EPD_RST: track 123.0 -> 109.9 mm, vias 3 -> 2
- net RX: track 9.90 -> 22.1 mm
- net TX: track 10.8 -> 21.7 mm
- net VBUS: track 70.7 -> 80.8 mm
- net N$8: track 17.0 -> 25.3 mm, vias 2 -> 0
- net USB_D-: track 147.9 -> 141.0 mm
- net FLASH_CS: track 51.1 -> 57.4 mm, vias 2 -> 3
- net MOSI: track 187.7 -> 181.4 mm, vias 6 -> 2
- net N$17: track 10.0 -> 3.98 mm
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
Commit message: Incarcare versiuni finale PCB (2D si 3D)
Parts:
- removed TP1, TP10, TP11, TP12, TP13, TP16, TP17, TP2, TP5, TP6, TP7, TP8, TP9: TPTP20R, DeskAssistant v19 v1:TP20R
- added 3V3, EPD_3V3, EPD_3V3_C, EPD_BUSY, EPD_CS, EPD_DC, EPD_RST, GND, MISO, MOSI, RX, SCK, TX: TPTP20R, DeskAssistant v19 v1:TP20R
- moved TP4 56.2 mm to (84.3, 96.0)
- moved TP15 36.6 mm to (84.1, 87.7)
- moved D9 25.5 mm to (31.3, 41.4)
- moved R5 25.5 mm to (33.3, 41.4)
- moved D12 21.2 mm to (46.2, 22.9)
- moved R8 21.1 mm to (44.4, 22.9)
- moved D10 19.9 mm to (38.5, 23.3)
- moved R6 16.8 mm to (40.5, 23.3)
- moved R2-PINH1 16.8 mm to (93.3, 55.5), turned to 90 degrees
- moved D11 15.6 mm to (52.8, 22.9)
- moved R7 15.4 mm to (50.2, 22.8)
- moved TP14 14.9 mm to (125.3, 65.2)
- moved C11 14.7 mm to (89.2, 39.8)
- moved C_DELAY 11.2 mm to (51.1, 100.8)
- moved IC1 11.0 mm to (48.3, 101.2)
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Connections:
- net 3V3: now also 3V3.TP; no longer TP16.TP
- net EPD_3V3: now also EPD_3V3.TP; no longer TP17.TP
- net EPD_3V3_C: now also EPD_3V3_C.TP; no longer TP13.TP
- net EPD_BUSY: now also EPD_BUSY.TP; no longer TP9.TP
- net EPD_CS: now also EPD_CS.TP; no longer TP10.TP
- net EPD_DC: now also EPD_DC.TP; no longer TP11.TP
- net EPD_RST: now also EPD_RST.TP; no longer TP12.TP
- net GND: now also GND.TP; no longer TP5.TP
- net MISO: now also MISO.TP; no longer TP6.TP
- net MOSI: now also MOSI.TP; no longer TP7.TP
- net RX: now also RX.TP; no longer TP2.TP
- net SCK: now also SCK.TP; no longer TP8.TP
- net TX: now also TX.TP; no longer TP1.TP
Routing:
- net EPD_3V3_C: track 158.3 -> 71.7 mm, vias 3 -> 0
- net EPD_CS: track 163.0 -> 104.7 mm, vias 5 -> 4
- net EPD_DC: track 170.8 -> 122.5 mm, vias 3 -> 0
- net SCK: track 155.7 -> 192.1 mm, vias 6 -> 2
- net FLASH_CS: track 57.4 -> 27.9 mm, vias 3 -> 2
- net EPD_3V3: track 35.7 -> 62.6 mm
- net RX: track 22.1 -> 6.09 mm
- net TX: track 21.7 -> 6.58 mm
- net EPD_RST: track 109.9 -> 124.4 mm
- net 3V3: track 388.6 -> 402.7 mm, vias 11 -> 15
- net DP: track 9.84 -> 21.6 mm, vias 2 -> 0
- net VBUS: track 80.8 -> 91.3 mm, vias 2 -> 0
- net EPD_BUSY: track 105.1 -> 115.6 mm, vias 2 -> 4
- net 32KHZ: track 91.8 -> 82.3 mm, vias 3 -> 2
- net N$8: track 25.3 -> 17.0 mm, vias 0 -> 2
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